File: VIM_2.1.sch (KiCad schematic (older format))
At the start: 13 parts, among them J1 BARREL_JACK, J2 Sliding switch, U14 LD1117, U8 lm2596 - 5v, U9 LD1117S33CTR

Commit message: added shivam changes text
Other:
- note added: "VIM"
- note added: "shivam changes\n"
- note added: "sushil changes"
- note removed: "ublox m8u"
Changed lines of the file:
@@
 $EndComp
 Text Notes 1750 3900 0    118  ~ 0
-ublox m8u
+VIM
 $Comp
 L +12V #PWR09
@@
 	5110 3900 5110 3690
 Connection ~ 5110 3690
+Text Notes 3580 5890 0    315  ~ 0
+sushil changes
+Text Notes 3550 6300 0    315  ~ 0
+shivam changes\n
 $EndSCHEMATC

Commit message: changes to b
Other:
- note added: "BANter\n\n"
Changed lines of the file:
@@
 LIBS:mpu
 LIBS:68 PIN
-LIBS:reugulators
 LIBS:simcard
 LIBS:j502
@@
 Text Notes 3550 6300 0    315  ~ 0
 shivam changes\n
+Text Notes 3650 7250 0    315  ~ 0
+BANter\n\n
 $EndSCHEMATC

Commit message: Revert "changes to b"
This reverts commit 29845ce44828af67f545c5cae162d888299830da.
Other:
- note removed: "BANter\n\n"
Changed lines of the file:
@@
 LIBS:mpu
 LIBS:68 PIN
+LIBS:reugulators
 LIBS:simcard
 LIBS:j502
@@
 Text Notes 3550 6300 0    315  ~ 0
 shivam changes\n
-Text Notes 3650 7250 0    315  ~ 0
-BANter\n\n
 $EndSCHEMATC
