File: VIM_2.1.sch (KiCad schematic (older format))
At the start: 13 parts, among them J1 BARREL_JACK, J2 Sliding switch, U14 LD1117, U8 lm2596 - 5v, U9 LD1117S33CTR

Commit message: update
Other:
- note added: "VIM"
- note removed: "ublox m8u"
Changed lines of the file:
@@
 $EndComp
 Text Notes 1750 3900 0    118  ~ 0
-ublox m8u
+VIM
 $Comp
 L +12V #PWR09

Commit message: pcb print 28 jul
Parts:
- C17: footprint Capacitors_THT:CP_Radial_D5.0mm_P2.50mm -> Capacitors_SMD:CP_Elec_8x6.7
- C19: footprint Capacitors_THT:CP_Radial_D5.0mm_P2.50mm -> Capacitors_SMD:CP_Elec_6.3x5.7
- L1: footprint Inductors_THT:L_Radial_D7.0mm_P3.00mm -> Inductors_SMD:L_7.3x7.3_H3.5
Changed lines of the file:
@@
 LIBS:mpu
 LIBS:68 PIN
-LIBS:reugulators
 LIBS:simcard
 LIBS:j502
@@
 F 0 "L1" V 4800 4100 50  0000 C CNN
 F 1 "68uH" V 4750 4250 50  0000 C CNN
-F 2 "Inductors_THT:L_Radial_D7.0mm_P3.00mm" H 4850 4100 50  0001 C CNN
+F 2 "Inductors_SMD:L_7.3x7.3_H3.5" H 4850 4100 50  0001 C CNN
 F 3 "" H 4850 4100 50  0001 C CNN
 	1    4850 4100
@@
 F 0 "C19" H 5525 4800 50  0000 L CNN
 F 1 "220uF" H 5525 4600 50  0000 L CNN
-F 2 "Capacitors_THT:CP_Radial_D5.0mm_P2.50mm" H 5500 4700 50  0001 C CNN
+F 2 "Capacitors_SMD:CP_Elec_6.3x5.7" H 5500 4700 50  0001 C CNN
 F 3 "" H 5500 4700 50  0001 C CNN
 	1    5500 4700
@@
 F 0 "C17" H 4325 4700 50  0000 L CNN
 F 1 "47uF" H 4325 4500 50  0000 L CNN
-F 2 "Capacitors_THT:CP_Radial_D5.0mm_P2.50mm" H 4300 4600 50  0001 C CNN
+F 2 "Capacitors_SMD:CP_Elec_8x6.7" H 4300 4600 50  0001 C CNN
 F 3 "" H 4300 4600 50  0001 C CNN
 	1    4300 4600
