File: file5AF7AEF3.sch (KiCad schematic (older format))
At the start: 13 parts, among them Q5 Q_NPN_BEC, U18 ufl, U19 ublox_m8u

Commit message: update
Parts:
- U19: value ublox_m8u -> vim
Changed lines of the file:
@@
 P 5600 2800
 F 0 "U19" H 5600 3650 60  0000 C CNN
-F 1 "ublox_m8u" H 5600 2150 60  0000 C CNN
+F 1 "vim" H 5600 2150 60  0000 C CNN
 F 2 "ublox:MU8" H 5600 2800 60  0001 C CNN
 F 3 "" H 5600 2800 60  0001 C CNN
