File: EMMC.sch (KiCad schematic (older format))
At the start: 1 part, among them U10 emmc

Commit message: Final pcb given to pcbpower
fleet management vim with following features
- ublox m8u, mc60
- mpu6050
- vibration sensor
- buzzer, switches, thottle bypass,
- sim interface according to quectel
Parts:
- U10: footprint emmc1:eMMC1 -> emmc1:eMMC2.4
Changed lines of the file:
@@
 LIBS:mpu
 LIBS:68 PIN
+LIBS:reugulators
 LIBS:simcard
 LIBS:j502
@@
 F 0 "U10" H 6150 950 60  0000 C CNN
 F 1 "emmc" H 6000 2250 60  0000 C CNN
-F 2 "emmc1:eMMC1" H 5050 2250 60  0001 C CNN
+F 2 "emmc1:eMMC2.4" H 5050 2250 60  0001 C CNN
 F 3 "" H 5050 2250 60  0001 C CNN
 	1    5050 2250
@@
 Connection ~ 4450 3950
 $Comp
-L +1V8 #PWR039
+L +1V8 #PWR040
 U 1 1 59EEFE16
 P 4250 3950
-F 0 "#PWR039" H 4250 3800 50  0001 C CNN
+F 0 "#PWR040" H 4250 3800 50  0001 C CNN
 F 1 "+1V8" H 4250 4090 50  0000 C CNN
 F 2 "" H 4250 3950 50  0001 C CNN
@@
 $EndComp
 $Comp
-L +3.3V #PWR040
+L +3.3V #PWR041
 U 1 1 59EEFE2C
 P 4250 3600
-F 0 "#PWR040" H 4250 3450 50  0001 C CNN
+F 0 "#PWR041" H 4250 3450 50  0001 C CNN
 F 1 "+3.3V" H 4250 3740 50  0000 C CNN
 F 2 "" H 4250 3600 50  0001 C CNN
@@
 $EndComp
 $Comp
-L GND #PWR041
+L GND #PWR042
 U 1 1 59EEFE56
 P 4250 3300
-F 0 "#PWR041" H 4250 3050 50  0001 C CNN
+F 0 "#PWR042" H 4250 3050 50  0001 C CNN
 F 1 "GND" H 4250 3150 50  0000 C CNN
 F 2 "" H 4250 3300 50  0001 C CNN
@@
 $EndComp
 $Comp
-L GND #PWR042
+L GND #PWR043
 U 1 1 59EEFE6C
 P 4250 3000
-F 0 "#PWR042" H 4250 2750 50  0001 C CNN
+F 0 "#PWR043" H 4250 2750 50  0001 C CNN
 F 1 "GND" H 4250 2850 50  0000 C CNN
 F 2 "" H 4250 3000 50  0001 C CNN
