File: file5986FC30.sch (KiCad schematic (older format))
At the start: 55 parts, among them Q1 Q_NPN_BEC, Q2 Q_NPN_BEC, Q3 Q_NPN_BEC, Q4 Q_NPN_BEC, U12 CM1224, U15 ufl, U17 ufl, U3 MIC29302, U5 J502, U6 AP131-33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

Commit message: final
Parts:
- AE1: footprint chip antenna:chip antenaa -> ANTENNASMD:bluetooth_antenna
Changed lines of the file:
@@
 SIM1_DATA
 $Comp
-L GND #PWR017
+L GND #PWR27
 U 1 1 598AB1C6
 P 3450 6050
-F 0 "#PWR017" H 3450 5800 50  0001 C CNN
+F 0 "#PWR27" H 3450 5800 50  0001 C CNN
 F 1 "GND" H 3450 5900 50  0000 C CNN
 F 2 "" H 3450 6050 50  0000 C CNN
@@
 $EndComp
 $Comp
-L GND #PWR018
+L GND #PWR22
 U 1 1 598AB649
 P 2350 1350
-F 0 "#PWR018" H 2350 1100 50  0001 C CNN
+F 0 "#PWR22" H 2350 1100 50  0001 C CNN
 F 1 "GND" H 2350 1200 50  0000 C CNN
 F 2 "" H 2350 1350 50  0000 C CNN
@@
 $EndComp
 $Comp
-L GND #PWR019
+L GND #PWR24
 U 1 1 598AB77B
 P 2850 1500
-F 0 "#PWR019" H 2850 1250 50  0001 C CNN
+F 0 "#PWR24" H 2850 1250 50  0001 C CNN
 F 1 "GND" H 2850 1350 50  0000 C CNN
 F 2 "" H 2850 1500 50  0000 C CNN
@@
 $EndComp
 $Comp
-L GND #PWR020
+L GND #PWR25
 U 1 1 598AB798
 P 3300 1500
-F 0 "#PWR020" H 3300 1250 50  0001 C CNN
+F 0 "#PWR25" H 3300 1250 50  0001 C CNN
 F 1 "GND" H 3300 1350 50  0000 C CNN
 F 2 "" H 3300 1500 50  0000 C CNN
@@
 $EndComp
 $Comp
-L GND #PWR021
+L GND #PWR20
 U 1 1 598AC537
 P 2200 2250
-F 0 "#PWR021" H 2200 2000 50  0001 C CNN
+F 0 "#PWR20" H 2200 2000 50  0001 C CNN
 F 1 "GND" H 2200 2100 50  0000 C CNN
 F 2 "" H 2200 2250 50  0000 C CNN
@@
 $EndComp
 $Comp
-L GND #PWR022
+L GND #PWR31
 U 1 1 598AD3DF
 P 5250 1500
-F 0 "#PWR022" H 5250 1250 50  0001 C CNN
+F 0 "#PWR31" H 5250 1250 50  0001 C CNN
 F 1 "GND" H 5250 1350 50  0000 C CNN
 F 2 "" H 5250 1500 50  0000 C CNN
@@
 vbat
 $Comp
-L GND #PWR023
+L GND #PWR32
 U 1 1 598BD80C
 P 5650 5400
-F 0 "#PWR023" H 5650 5150 50  0001 C CNN
+F 0 "#PWR32" H 5650 5150 50  0001 C CNN
 F 1 "GND" H 5650 5250 50  0000 C CNN
 F 2 "" H 5650 5400 50  0000 C CNN
@@
 $EndComp
 $Comp
-L GND #PWR024
+L GND #PWR33
 U 1 1 598BD946
 P 5650 5800
-F 0 "#PWR024" H 5650 5550 50  0001 C CNN
+F 0 "#PWR33" H 5650 5550 50  0001 C CNN
 F 1 "GND" H 5650 5650 50  0000 C CNN
 F 2 "" H 5650 5800 50  0000 C CNN
@@
 $EndComp
 $Comp
-L GND #PWR025
+L GND #PWR34
 U 1 1 598BE202
 P 5650 6050
-F 0 "#PWR025" H 5650 5800 50  0001 C CNN
+F 0 "#PWR34" H 5650 5800 50  0001 C CNN
 F 1 "GND" H 5650 5900 50  0000 C CNN
 F 2 "" H 5650 6050 50  0000 C CNN
@@
 GNSS_VCC_EN
 $Comp
-L GND #PWR026
+L GND #PWR26
 U 1 1 598C63D5
 P 3450 4750
-F 0 "#PWR026" H 3450 4500 50  0001 C CNN
+F 0 "#PWR26" H 3450 4500 50  0001 C CNN
 F 1 "GND" H 3450 4600 50  0000 C CNN
 F 2 "" H 3450 4750 50  0000 C CNN
@@
 $EndComp
 $Comp
-L GND #PWR027
+L GND #PWR38
 U 1 1 59931901
 P 8350 2400
-F 0 "#PWR027" H 8350 2150 50  0001 C CNN
+F 0 "#PWR38" H 8350 2150 50  0001 C CNN
 F 1 "GND" H 8350 2250 50  0000 C CNN
 F 2 "" H 8350 2400 50  0001 C CNN
@@
 $EndComp
 $Comp
-L GND #PWR028
+L GND #PWR39
 U 1 1 59933041
 P 10550 2150
-F 0 "#PWR028" H 10550 1900 50  0001 C CNN
+F 0 "#PWR39" H 10550 1900 50  0001 C CNN
 F 1 "GND" H 10550 2000 50  0000 C CNN
 F 2 "" H 10550 2150 50  0001 C CNN
@@
 $EndComp
 $Comp
-L GND #PWR029
+L GND #PWR29
 U 1 1 599B1446
 P 3700 7450
-F 0 "#PWR029" H 3700 7200 50  0001 C CNN
+F 0 "#PWR29" H 3700 7200 50  0001 C CNN
 F 1 "GND" H 3700 7300 50  0000 C CNN
 F 2 "" H 3700 7450 50  0000 C CNN
@@
 $EndComp
 $Comp
-L GND #PWR030
+L GND #PWR28
 U 1 1 5994F897
 P 3550 6450
-F 0 "#PWR030" H 3550 6200 50  0001 C CNN
+F 0 "#PWR28" H 3550 6200 50  0001 C CNN
 F 1 "GND" H 3550 6300 50  0000 C CNN
 F 2 "" H 3550 6450 50  0001 C CNN
@@
 GNSS_VCC
 $Comp
-L GND #PWR031
+L GND #PWR35
 U 1 1 59974B9B
 P 6000 3900
-F 0 "#PWR031" H 6000 3650 50  0001 C CNN
+F 0 "#PWR35" H 6000 3650 50  0001 C CNN
 F 1 "GND" H 6000 3750 50  0000 C CNN
 F 2 "" H 6000 3900 50  0001 C CNN
@@
 $EndComp
 $Comp
-L GND #PWR032
+L GND #PWR21
 U 1 1 5997C38C
 P 2300 3650
-F 0 "#PWR032" H 2300 3400 50  0001 C CNN
+F 0 "#PWR21" H 2300 3400 50  0001 C CNN
 F 1 "GND" H 2300 3500 50  0000 C CNN
 F 2 "" H 2300 3650 50  0001 C CNN
@@
 vbat
 $Comp
-L GND #PWR033
+L GND #PWR36
 U 1 1 599838C3
 P 6450 5800
-F 0 "#PWR033" H 6450 5550 50  0001 C CNN
+F 0 "#PWR36" H 6450 5550 50  0001 C CNN
 F 1 "GND" H 6450 5650 50  0000 C CNN
 F 2 "" H 6450 5800 50  0000 C CNN
@@
 regulatorIN
 $Comp
-L GND #PWR034
+L GND #PWR17
 U 1 1 599DFD1C
 P 1450 1550
-F 0 "#PWR034" H 1450 1300 50  0001 C CNN
+F 0 "#PWR17" H 1450 1300 50  0001 C CNN
 F 1 "GND" H 1450 1400 50  0000 C CNN
 F 2 "" H 1450 1550 50  0000 C CNN
@@
 GNSS_VCC
 $Comp
-L GND #PWR035
+L GND #PWR18
 U 1 1 59A6620C
 P 1550 6150
-F 0 "#PWR035" H 1550 5900 50  0001 C CNN
+F 0 "#PWR18" H 1550 5900 50  0001 C CNN
 F 1 "GND" H 1550 6000 50  0000 C CNN
 F 2 "" H 1550 6150 50  0001 C CNN
@@
 $EndComp
 $Comp
-L GND #PWR036
+L GND #PWR23
 U 1 1 5AC60895
 P 2800 5750
-F 0 "#PWR036" H 2800 5500 50  0001 C CNN
+F 0 "#PWR23" H 2800 5500 50  0001 C CNN
 F 1 "GND" H 2850 5600 50  0000 C CNN
 F 2 "" H 2800 5750 50  0000 C CNN
@@
 NoConn ~ 5200 6550
 $Comp
-L GND #PWR037
+L GND #PWR37
 U 1 1 5ACB6823
 P 7400 6150
-F 0 "#PWR037" H 7400 5900 50  0001 C CNN
+F 0 "#PWR37" H 7400 5900 50  0001 C CNN
 F 1 "GND" H 7400 6000 50  0000 C CNN
 F 2 "" H 7400 6150 50  0000 C CNN
@@
 $EndComp
 $Comp
-L GND #PWR038
+L GND #PWR19
 U 1 1 5ACBBEA3
 P 2150 4650
-F 0 "#PWR038" H 2150 4400 50  0001 C CNN
+F 0 "#PWR19" H 2150 4400 50  0001 C CNN
 F 1 "GND" H 2150 4500 50  0000 C CNN
 F 2 "" H 2150 4650 50  0000 C CNN
@@
 	3900 2050 3900 2150
 $Comp
-L GND #PWR039
+L GND #PWR30
 U 1 1 5B1E55C6
 P 3900 2150
-F 0 "#PWR039" H 3900 1900 50  0001 C CNN
+F 0 "#PWR30" H 3900 1900 50  0001 C CNN
 F 1 "GND" H 3900 2000 50  0000 C CNN
 F 2 "" H 3900 2150 50  0000 C CNN
@@
 F 0 "AE1" H 1975 6625 50  0000 R CNN
 F 1 "Antenna" H 1975 6550 50  0000 R CNN
-F 2 "chip antenna:chip antenaa" H 2050 6550 50  0001 C CNN
+F 2 "ANTENNASMD:bluetooth_antenna" H 2050 6550 50  0001 C CNN
 F 3 "" H 2050 6550 50  0001 C CNN
 	1    2050 6550
