File: file59818FC9.sch (KiCad schematic (older format))
At the start: 76 parts, among them J10 Conn_01x03, J3 Conn_01x05, J4 Conn_01x03, J5 uart, J6 Conn_01x03, J8 Conn_01x03, J9 Conn_01x03, P1 USB_OTG, P2 charging, Q10 Q_NPN_BEC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

Commit message: PCB SENT TO PCB POWER
Parts:
- gave numbers to parts that had none: 1
Connections:
- net a: now also J7.4 (P4)
- net b: now also J7.3 (P3)
- net charging: now also U1.10 (PC2); no longer U1.9 (PC1)
- net in4: now also U1.8 (PC0); no longer U1.7 (NRST)
- net in5: now also U1.9 (PC1); no longer U1.8 (PC0)
